File: pcm5102dac.brd (EAGLE design)
At the start: 39.6 x 22.6 mm, 23 parts

Commit message: v1.1
Parts:
- added U$4: GND_CONNECT, SparkFun-Passives:GND_CONNECT
- moved C1 5.14 mm to (31.5, 21.6)
Connections:
- net AGND: now also U$4.2
- net DGND: now also U$4.1
Changed lines of the file:
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@@
 <element name="C12" library="SparkFun-Capacitors" package="0805" value="" x="29.464" y="25.908" rot="R90"/>
 <element name="C13" library="SparkFun-Capacitors" package="0805" value="" x="27.94" y="25.908" rot="R90"/>
-<element name="C1" library="SparkFun-Capacitors" package="0805" value="" x="36.322" y="19.812" rot="R90"/>
+<element name="C1" library="SparkFun-Capacitors" package="0805" value="" x="31.496" y="21.59" rot="R90"/>
 <element name="C2" library="SparkFun-Capacitors" package="0805" value="" x="28.702" y="21.59" rot="R90"/>
 <element name="C3" library="SparkFun-Capacitors" package="0805" value="" x="25.654" y="23.114" smashed="yes" rot="R270">
@@
 <attribute name="VALUE" x="37.338" y="15.621" size="1.27" layer="28" rot="MR270"/>
 </element>
+<element name="U$4" library="SparkFun-Passives" package="GND_CONNECT" value="GND_CONNECT" x="26.416" y="33.528" smashed="yes" rot="R90"/>
 </elements>
 <signals>
@@
 <contactref element="C3" pad="1"/>
 <contactref element="U$1" pad="1"/>
-<wire x1="36.322" y1="19.05" x2="36.83" y2="19.05" width="0.254" layer="1"/>
-<wire x1="36.322" y1="19.05" x2="36.322" y2="18.912" width="0.254" layer="1"/>
-<wire x1="38.1" y1="17.78" x2="36.83" y2="19.05" width="0.4064" layer="1"/>
-<wire x1="39.522" y1="17.78" x2="38.1" y2="17.78" width="0.4064" layer="1"/>
-<wire x1="36.83" y1="19.05" x2="36.322" y2="18.912" width="0.254" layer="1"/>
-<wire x1="25.654" y1="24.014" x2="25.654" y2="24.3832" width="0.4064" layer="1"/>
-<wire x1="25.654" y1="24.3832" x2="26.2858" y2="25.015" width="0.4064" layer="1"/>
+<wire x1="25.654" y1="24.014" x2="25.4" y2="23.8752" width="0.4064" layer="1"/>
+<wire x1="25.4" y1="23.8752" x2="26.2858" y2="25.015" width="0.4064" layer="1"/>
 <wire x1="24.776" y1="20.69" x2="24.384" y2="21.082" width="0.4064" layer="1"/>
 <wire x1="24.384" y1="21.082" x2="24.384" y2="24.13" width="0.4064" layer="1"/>
@@
 <wire x1="26.1848" y1="29.464" x2="26.2858" y2="29.565" width="0.3048" layer="1"/>
 <wire x1="24.892" y1="29.464" x2="24.384" y2="28.956" width="0.3048" layer="1"/>
-<wire x1="25.654" y1="24.3832" x2="24.6372" y2="24.3832" width="0.4064" layer="1"/>
-<wire x1="24.6372" y1="24.3832" x2="24.384" y2="24.13" width="0.4064" layer="1"/>
+<wire x1="25.4" y1="23.8752" x2="24.6372" y2="23.8752" width="0.4064" layer="1"/>
+<wire x1="24.6372" y1="23.8752" x2="24.384" y2="24.13" width="0.4064" layer="1"/>
 <wire x1="24.776" y1="20.69" x2="28.702" y2="20.69" width="0.4064" layer="1"/>
-<wire x1="34.682" y1="20.69" x2="28.702" y2="20.69" width="0.4064" layer="1"/>
-<wire x1="34.682" y1="20.69" x2="35.052" y2="20.32" width="0.4064" layer="1"/>
-<wire x1="35.052" y1="20.32" x2="35.052" y2="19.304" width="0.4064" layer="1"/>
-<wire x1="35.052" y1="19.304" x2="35.306" y2="19.05" width="0.4064" layer="1"/>
-<wire x1="35.306" y1="19.05" x2="36.184" y2="19.05" width="0.4064" layer="1"/>
-<wire x1="36.184" y1="19.05" x2="36.322" y2="18.912" width="0.4064" layer="1"/>
+<wire x1="39.522" y1="17.78" x2="36.83" y2="17.78" width="0.4064" layer="1"/>
+<wire x1="36.83" y1="17.78" x2="35.56" y2="19.05" width="0.4064" layer="1"/>
+<wire x1="35.56" y1="19.05" x2="35.56" y2="20.066" width="0.4064" layer="1"/>
+<wire x1="35.56" y1="20.066" x2="34.798" y2="20.828" width="0.4064" layer="1"/>
+<wire x1="34.798" y1="20.828" x2="31.612" y2="20.828" width="0.4064" layer="1"/>
+<wire x1="31.612" y1="20.828" x2="31.496" y2="20.69" width="0.4064" layer="1"/>
+<wire x1="31.496" y1="20.69" x2="28.702" y2="20.69" width="0.4064" layer="1"/>
 </signal>
 <signal name="N$11">
@@
 <wire x1="20.4502" y1="25.665" x2="19.177" y2="25.665" width="0.254" layer="1"/>
 <wire x1="19.177" y1="25.665" x2="18.796" y2="26.046" width="0.254" layer="1"/>
-<via x="19.304" y="22.86" extent="1-16" drill="0.6"/>
+<via x="19.05" y="22.86" extent="1-16" drill="0.6"/>
 <via x="27.686" y="18.796" extent="1-16" drill="0.6"/>
 <polygon width="0.254" layer="16" isolate="0.4064">
@@
 <wire x1="21.336" y1="34.163" x2="23.749" y2="34.163" width="0.254" layer="1"/>
 <wire x1="23.749" y1="34.163" x2="23.876" y2="34.036" width="0.254" layer="1"/>
-<via x="25.654" y="32.512" extent="1-16" drill="0.6"/>
-<via x="21.59" y="27.686" extent="1-16" drill="0.6"/>
+<via x="24.638" y="32.004" extent="1-16" drill="0.6"/>
+<via x="21.59" y="27.686" extent="1-16" drill="0.6" diameter="0.3048"/>
 <via x="27.686" y="14.224" extent="1-16" drill="0.6"/>
 <via x="27.686" y="16.51" extent="1-16" drill="0.6"/>
 <contactref element="U$3" pad="1"/>
+<contactref element="U$4" pad="1"/>
 </signal>
 <signal name="DVCC">
@@
 <via x="25.146" y="26.416" extent="1-16" drill="0.3302"/>
 <via x="27.178" y="22.352" extent="1-16" drill="0.6"/>
-<via x="36.322" y="22.606" extent="1-16" drill="0.6"/>
+<via x="39.624" y="22.098" extent="1-16" drill="0.6"/>
 <contactref element="C6" pad="2"/>
 <via x="36.83" y="13.97" extent="1-16" drill="0.6"/>
@@
 <wire x1="26.162" y1="30.226" x2="26.2858" y2="30.215" width="0.254" layer="1"/>
 <wire x1="23.876" y1="27.94" x2="23.876" y2="27.817909375" width="0.254" layer="1"/>
-<via x="30.988" y="23.876" extent="1-16" drill="0.6"/>
+<via x="29.972" y="23.622" extent="1-16" drill="0.6"/>
 <wire x1="26.162" y1="30.226" x2="27.686" y2="30.226" width="0.4064" layer="1"/>
 <wire x1="26.162" y1="30.226" x2="23.622" y2="30.226" width="0.4064" layer="1"/>
@@
 <via x="36.83" y="16.002" extent="1-16" drill="0.6"/>
 <via x="42.672" y="20.066" extent="1-16" drill="0.6"/>
-<via x="39.624" y="22.606" extent="1-16" drill="0.6"/>
+<via x="37.338" y="20.066" extent="1-16" drill="0.6"/>
 <contactref element="U$3" pad="2"/>
+<contactref element="U$4" pad="2"/>
 </signal>
 </signals>
