File: pcm5102dac.sch (EAGLE design)
At the start: 23 parts

Commit message: v1.1
Parts:
- added U$4: GND_CONNECT, SparkFun-Passives:GND_CONNECT
Connections:
- net AGND: now also U$4.AGND
- net DGND: now also U$4.DGND
Changed lines of the file:
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@@
 <part name="C6" library="SparkFun-Capacitors" deviceset="CAP" device="0805"/>
 <part name="U$3" library="SparkFun-Passives" deviceset="GND_CONNECT" device=""/>
+<part name="U$4" library="SparkFun-Passives" deviceset="GND_CONNECT" device=""/>
 </parts>
 <sheets>
@@
 <instance part="C6" gate="G$1" x="-48.26" y="132.08"/>
 <instance part="U$3" gate="G$1" x="-35.56" y="106.68" rot="R90"/>
+<instance part="U$4" gate="G$1" x="78.74" y="134.62" rot="R90"/>
 </instances>
 <busses>
@@
 <pinref part="VREG1" gate="VREG" pin="VOUT"/>
 <wire x1="-25.4" y1="137.16" x2="-17.78" y2="137.16" width="0.1524" layer="91"/>
+<label x="-22.86" y="137.16" size="1.778" layer="95"/>
 </segment>
 <segment>
@@
 <pinref part="U$1" gate="G$1" pin="CPVDD"/>
 <wire x1="38.1" y1="83.82" x2="48.26" y2="83.82" width="0.1524" layer="91"/>
-<wire x1="7.62" y1="86.36" x2="2.54" y2="86.36" width="0.1524" layer="91"/>
+<label x="22.86" y="88.9" size="1.778" layer="95"/>
 </segment>
 <segment>
@@
 <wire x1="30.48" y1="55.88" x2="17.78" y2="55.88" width="0.1524" layer="91"/>
 <wire x1="17.78" y1="55.88" x2="15.24" y2="55.88" width="0.1524" layer="91"/>
+<label x="10.16" y="55.88" size="1.778" layer="95"/>
 </segment>
 </net>
@@
 <wire x1="27.94" y1="78.74" x2="22.86" y2="78.74" width="0.1524" layer="91"/>
 <pinref part="U$1" gate="G$1" pin="CPGND"/>
+<label x="20.32" y="81.28" size="1.778" layer="95"/>
 </segment>
 <segment>
@@
 <pinref part="U$1" gate="G$1" pin="AGND"/>
 <wire x1="43.18" y1="55.88" x2="48.26" y2="55.88" width="0.1524" layer="91"/>
+<label x="10.16" y="45.72" size="1.778" layer="95"/>
 </segment>
 <segment>
@@
 <wire x1="-43.18" y1="116.84" x2="-43.18" y2="124.46" width="0.1524" layer="91"/>
 <pinref part="U$3" gate="G$1" pin="AGND"/>
+<wire x1="-17.78" y1="129.54" x2="-12.7" y2="129.54" width="0.1524" layer="91"/>
+<wire x1="-12.7" y1="129.54" x2="-12.7" y2="154.94" width="0.1524" layer="91"/>
+<pinref part="U$4" gate="G$1" pin="AGND"/>
+<wire x1="71.12" y1="144.78" x2="71.12" y2="154.94" width="0.1524" layer="91"/>
+<wire x1="-12.7" y1="154.94" x2="71.12" y2="154.94" width="0.1524" layer="91"/>
 </segment>
 </net>
@@
 <pinref part="JP2" gate="G$1" pin="5"/>
 <wire x1="134.62" y1="76.2" x2="129.54" y2="76.2" width="0.1524" layer="91"/>
+<label x="127" y="76.2" size="1.778" layer="95"/>
 </segment>
 </net>
@@
 <pinref part="JP2" gate="G$1" pin="6"/>
 <wire x1="134.62" y1="73.66" x2="129.54" y2="73.66" width="0.1524" layer="91"/>
+<label x="127" y="73.66" size="1.778" layer="95"/>
 </segment>
 </net>
@@
 <pinref part="JP2" gate="G$1" pin="3"/>
 <wire x1="134.62" y1="81.28" x2="129.54" y2="81.28" width="0.1524" layer="91"/>
+<label x="127" y="81.28" size="1.778" layer="95"/>
 </segment>
 </net>
@@
 <pinref part="JP2" gate="G$1" pin="4"/>
 <wire x1="134.62" y1="78.74" x2="129.54" y2="78.74" width="0.1524" layer="91"/>
+<label x="127" y="78.74" size="1.778" layer="95"/>
 </segment>
 </net>
@@
 <wire x1="-48.26" y1="137.16" x2="-55.88" y2="137.16" width="0.1524" layer="91"/>
 <junction x="-48.26" y="137.16"/>
+<label x="-55.88" y="137.16" size="1.778" layer="95"/>
 </segment>
 <segment>
@@
 <pinref part="VREG3" gate="VREG" pin="VIN"/>
 <wire x1="0" y1="137.16" x2="-7.62" y2="137.16" width="0.1524" layer="91"/>
+<label x="-7.62" y="137.16" size="1.778" layer="95"/>
 </segment>
 <segment>
@@
 <pinref part="U$1" gate="G$1" pin="DGND"/>
 <wire x1="66.04" y1="81.28" x2="71.12" y2="81.28" width="0.1524" layer="91"/>
+<label x="88.9" y="83.82" size="1.778" layer="95"/>
 </segment>
 <segment>
@@
 <wire x1="-33.02" y1="116.84" x2="-30.48" y2="124.46" width="0.1524" layer="91"/>
 <pinref part="U$3" gate="G$1" pin="DGND"/>
+<wire x1="-7.62" y1="129.54" x2="0" y2="129.54" width="0.1524" layer="91"/>
+<wire x1="0" y1="129.54" x2="0" y2="114.3" width="0.1524" layer="91"/>
+<wire x1="0" y1="114.3" x2="22.86" y2="114.3" width="0.1524" layer="91"/>
+<wire x1="22.86" y1="114.3" x2="22.86" y2="147.32" width="0.1524" layer="91"/>
+<wire x1="22.86" y1="147.32" x2="76.2" y2="147.32" width="0.1524" layer="91"/>
+<wire x1="76.2" y1="147.32" x2="76.2" y2="152.4" width="0.1524" layer="91"/>
+<pinref part="U$4" gate="G$1" pin="DGND"/>
+<wire x1="81.28" y1="144.78" x2="81.28" y2="152.4" width="0.1524" layer="91"/>
+<wire x1="76.2" y1="152.4" x2="81.28" y2="152.4" width="0.1524" layer="91"/>
 </segment>
 <segment>
@@
 <pinref part="JP2" gate="G$1" pin="2"/>
 <wire x1="134.62" y1="83.82" x2="129.54" y2="83.82" width="0.1524" layer="91"/>
+<label x="127" y="83.82" size="1.778" layer="95"/>
 </segment>
 </net>
@@
 <pinref part="VREG3" gate="VREG" pin="VOUT"/>
 <wire x1="20.32" y1="137.16" x2="30.48" y2="137.16" width="0.1524" layer="91"/>
+<label x="30.48" y="137.16" size="1.778" layer="95"/>
 </segment>
 <segment>
@@
 <pinref part="JP2" gate="G$1" pin="1"/>
 <wire x1="134.62" y1="86.36" x2="129.54" y2="86.36" width="0.1524" layer="91"/>
+<label x="127" y="86.36" size="1.778" layer="95"/>
 </segment>
 <segment>
@@
 <pinref part="U$1" gate="G$1" pin="DVDD"/>
 <wire x1="66.04" y1="83.82" x2="71.12" y2="83.82" width="0.1524" layer="91"/>
-</segment>
-</net>
+<label x="88.9" y="91.44" size="1.778" layer="95"/>
+</segment>
+</net>
