File: PCM5102a.brd (EAGLE design)
At the start: 39.6 x 20.5 mm, 30 parts, among them U2 DVCC, U3 CPVDD, U4 AVDD

Commit message: V1.21
Parts:
- removed U$3: GND_CONNECT, SparkFun-Passives:GND_CONNECT
- moved C16 3.69 mm to (34.5, 31.8), turned to 90 degrees
- moved JP3 2.93 mm to (17.4, 31.4)
- moved U$2 2.44 mm to (23.5, 27.4)
- moved C7 0.30 mm to (16.5, 17.4)
- moved C10 0.15 mm to (19.1, 24.2)
Connections:
- net AGND: no longer U$3.2
- net DGND: no longer U$3.1
Routing:
- net AGND: track 73.4 -> 50.6 mm, vias 0 -> 6
- net DGND: track 35.9 -> 16.8 mm, vias 0 -> 17
- net SCK: track 7.57 -> 4.11 mm
- net SCKI: track 6.55 -> 3.69 mm
- net CPGND: track 23.1 -> 21.1 mm, vias 1 -> 18
- net AVDD: track 13.4 -> 12.0 mm
- net DVCC: track 42.4 -> 43.4 mm
- net BCK: track 9.14 -> 8.34 mm
Other:
- board text added: "DVDD"
- board text added: "Filter latency"
- board text added: "Low"
- board text added: "Normal"
- board text removed: "FLT"
