File: PCM5102a.sch (EAGLE design)
At the start: 30 parts, among them U2 DVCC, U3 CPVDD, U4 AVDD

Commit message: V1.21
Parts:
- removed U$3: GND_CONNECT, SparkFun-Passives:GND_CONNECT
Connections:
- net AGND: no longer U$3.AGND
- net DGND: no longer U$3.DGND
Changed lines of the file:
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@@
 <part name="U$2" library="SparkFun-Passives" deviceset="GND_CONNECT" device=""/>
 <part name="JP2" library="SparkFun-Connectors" deviceset="M06" device="LOCK"/>
-<part name="U$3" library="SparkFun-Passives" deviceset="GND_CONNECT" device=""/>
 <part name="JP4" library="SparkFun-Connectors" deviceset="M02" device="LOCK" value="M02LOCK"/>
 <part name="U2" library="SparkFun-PowerIC" deviceset="V_REG_LDO" device="SMD" value="DVCC"/>
@@
 <instance part="U$2" gate="G$1" x="-10.16" y="116.84" rot="R90"/>
 <instance part="JP2" gate="G$1" x="139.7" y="81.28" rot="R180"/>
-<instance part="U$3" gate="G$1" x="-30.48" y="116.84" rot="R90"/>
 <instance part="JP4" gate="G$1" x="25.4" y="187.96"/>
 <instance part="U2" gate="G$1" x="55.88" y="139.7"/>
@@
 <label x="88.9" y="182.88" size="1.778" layer="95"/>
 </segment>
-<segment>
-<wire x1="-38.1" y1="127" x2="-38.1" y2="129.54" width="0.1524" layer="91"/>
-<pinref part="U$3" gate="G$1" pin="AGND"/>
-<label x="-38.1" y="129.54" size="1.778" layer="95"/>
-</segment>
 </net>
 <net name="LRCK" class="0">
@@
 <pinref part="U$2" gate="G$1" pin="DGND"/>
 <wire x1="-7.62" y1="127" x2="-7.62" y2="129.54" width="0.1524" layer="91"/>
-<wire x1="-27.94" y1="127" x2="-27.94" y2="129.54" width="0.1524" layer="91"/>
-<pinref part="U$3" gate="G$1" pin="DGND"/>
-<label x="-27.94" y="129.54" size="1.778" layer="95"/>
 <label x="-7.62" y="129.54" size="1.778" layer="95"/>
 </segment>
